Commit message: feat : 3D 모델링

File: mastering_ros_robot_description_pkg/urdf/seven_dof_arm.xacro (robot description, xacro)
@@ -6,5 +6,5 @@
     </material>
     <material name="Red">
-        <color rgba="0.8 0.0 0.0 1.0"/>
+        <color rgba="1.0 .0 0.0 1.0"/>
     </material>
     <material name="White">

File: mastering_ros_robot_description_pkg/urdf/seven_dof_arm_with_rgbd.xacro (robot description, xacro)
@@ -92,5 +92,5 @@
 	       <box size="1 1 0.02" />
       </geometry>
-      </collision>>
+      </collision>
   </link>
   <gazebo reference="bottom_link">
